File: UINIO-EVB-STM32L051K8.kicad_pcb (KiCad board)
At the start: 2 copper layers, 34.4 x 36.6 mm, 28 parts, among them J1 Conn_01x14_Male, J2 Conn_01x14_Male, J3 Conn_01x04_Male, SW1 SW_Push, SW2 SW_Push, U1 ME6211C33M5G-N, U2 W25Q128JVSSIQ, U3 STM32L051K8U6, Y1 Crystal_GND24

Commit message: Generate the gerbers.
Changed lines of the file:
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@@
   (net 37 "unconnected-(USB1-PadB5)")
   (net 38 "unconnected-(USB1-PadB8)")
-  (net 39 "Net-(USB1-PadA4B9)")
+  (net 39 "Net-(F1-Pad1)")
   (footprint "Resistor_SMD:R_0402_1005Metric" (layer "F.Cu")
     (at 164.63 99.03 180)
@@
     (property "Sheetname" "")
     (attr smd)
-    (fp_text reference "R3" (at 0.07 0.97) (layer "F.SilkS")
+    (fp_text reference "R3" (at 0.02 1.09) (layer "F.SilkS")
       (effects (font (size 0.8 0.8) (thickness 0.1)))
     )
@@
     (property "Sheetname" "")
     (attr smd)
-    (fp_text reference "F1" (at -2.832 0.09) (layer "F.SilkS")
+    (fp_text reference "F1" (at 2.82 0.08) (layer "F.SilkS")
       (effects (font (size 0.8 0.8) (thickness 0.1)))
     )
@@
     (fp_line (start -1.6 -0.8) (end 1.6 -0.8) (layer "F.Fab") (width 0.1))
     (pad "1" smd roundrect (at -1.4 0 90) (size 1.25 1.75) (layers "F.Cu" "F.Paste" "F.Mask") (roundrect_rratio 0.2)
-      (net 39 "Net-(USB1-PadA4B9)") (pintype "passive"))
+      (net 39 "Net-(F1-Pad1)") (pintype "passive"))
     (pad "2" smd roundrect (at 1.4 0 90) (size 1.25 1.75) (layers "F.Cu" "F.Paste" "F.Mask") (roundrect_rratio 0.2)
       (net 2 "/VDD_5V") (pintype "passive"))
@@
       (net 1 "GND") (pinfunction "GND") (pintype "input"))
     (pad "A4B9" smd rect (at -2.4 -2.481 180) (size 0.6 1.15) (layers "F.Cu" "F.Paste" "F.Mask")
-      (net 39 "Net-(USB1-PadA4B9)") (pinfunction "VBUS") (pintype "input"))
+      (net 39 "Net-(F1-Pad1)") (pinfunction "VBUS") (pintype "input"))
     (pad "A5" smd rect (at -1.25 -2.481 180) (size 0.3 1.15) (layers "F.Cu" "F.Paste" "F.Mask")
       (net 33 "unconnected-(USB1-PadA5)") (pinfunction "CC1") (pintype "input+no_connect"))
@@
       (net 1 "GND") (pinfunction "GND") (pintype "input"))
     (pad "B4A9" smd rect (at 2.4 -2.481 180) (size 0.6 1.15) (layers "F.Cu" "F.Paste" "F.Mask")
-      (net 39 "Net-(USB1-PadA4B9)") (pinfunction "VBUS") (pintype "input"))
+      (net 39 "Net-(F1-Pad1)") (pinfunction "VBUS") (pintype "input"))
     (pad "B5" smd rect (at 1.75 -2.481 180) (size 0.3 1.15) (layers "F.Cu" "F.Paste" "F.Mask")
       (net 37 "unconnected-(USB1-PadB5)") (pinfunction "CC2") (pintype "input+no_connect"))
@@
     (property "Sheetname" "")
     (attr smd)
-    (fp_text reference "D1" (at -2.19 0.02) (layer "F.SilkS")
+    (fp_text reference "D1" (at -2.08 0.11) (layer "F.SilkS")
       (effects (font (size 0.8 0.8) (thickness 0.1)))
     )
@@
     (property "材质" "X7R")
     (attr smd)
-    (fp_text reference "C2" (at -1.745 -0.1) (layer "F.SilkS")
+    (fp_text reference "C2" (at -1.694 0.057) (layer "F.SilkS")
       (effects (font (size 0.8 0.8) (thickness 0.1)))
     )
@@
     (property "材质" "X7R")
     (attr smd)
-    (fp_text reference "C1" (at -1.778 0) (layer "F.SilkS")
+    (fp_text reference "C1" (at -1.65 0.035) (layer "F.SilkS")
       (effects (font (size 0.8 0.8) (thickness 0.1)))
     )
@@
   (segment (start 147.09 98.649) (end 147.09 99.649) (width 0.5) (layer "F.Cu") (net 1))
   (segment (start 166.26 105.78) (end 166.24 105.76) (width 0.5) (layer "F.Cu") (net 1))
-  (segment (start 160.12 105.78) (end 159.17 106.73) (width 0.5) (layer "F.Cu") (net 1))
   (segment (start 167.3875 99.04) (end 170.4 99.04) (width 0.3) (layer "F.Cu") (net 1))
   (segment (start 148.907 99.93) (end 150.675 101.698) (width 0.5) (layer "F.Cu") (net 1))
   (segment (start 164.64 121.59) (end 164.64 122.45) (width 0.3) (layer "F.Cu") (net 1))
   (segment (start 150.675 97.498) (end 159.325 97.498) (width 0.5) (layer "F.Cu") (net 1))
-  (segment (start 159.17 106.73) (end 159.17 108.79) (width 0.5) (layer "F.Cu") (net 1))
+  (segment (start 161.78 105.78) (end 159.86 105.78) (width 0.5) (layer "F.Cu") (net 1))
   (segment (start 155.28 113.93) (end 155.28 113.32) (width 0.3) (layer "F.Cu") (net 1))
   (segment (start 162.39 124.18) (end 163.18 123.39) (width 0.3) (layer "F.Cu") (net 1))
   (segment (start 164.45 105.76) (end 164.43 105.78) (width 0.5) (layer "F.Cu") (net 1))
   (segment (start 168.74 105.78) (end 170.4 104.12) (width 0.5) (layer "F.Cu") (net 1))
+  (segment (start 159.17 106.47) (end 159.17 108.79) (width 0.5) (layer "F.Cu") (net 1))
   (segment (start 147.371 99.93) (end 148.907 99.93) (width 0.5) (layer "F.Cu") (net 1))
+  (segment (start 159.86 105.78) (end 159.17 106.47) (width 0.5) (layer "F.Cu") (net 1))
   (segment (start 164.6 123.39) (end 164.64 123.43) (width 0.3) (layer "F.Cu") (net 1))
   (segment (start 163.18 123.39) (end 164.6 123.39) (width 0.3) (layer "F.Cu") (net 1))
@@
   (segment (start 164.64 122.45) (end 164.64 123.43) (width 0.3) (layer "F.Cu") (net 1))
   (segment (start 150.675 97.498) (end 150.675 101.698) (width 0.5) (layer "F.Cu") (net 1))
-  (segment (start 161.78 105.78) (end 160.12 105.78) (width 0.5) (layer "F.Cu") (net 1))
   (segment (start 154.39 123.7) (end 154.39 124.49) (width 0.3) (layer "F.Cu") (net 1))
   (segment (start 158.2 102.46) (end 158.563 102.46) (width 0.5) (layer "F.Cu") (net 1))

Commit message: Everything was checked.
Parts:
- moved ? 1.56 mm to (148.9, 121.6)
Other:
- board text added: "PA13/SWDIO"
- board text added: "PA14/SWCLK"
- board text added: "UINIO-EVB-STM32L051K8"
- board text added: "VDD_3.3V"
- board text added: "Version 1.0.0"
- board text removed: "UINIO-EVB-STM32L051K8 Version 1.0.0"
Changed lines of the file:
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@@
       (layerselection 0x00010fc_ffffffff)
       (disableapertmacros false)
-      (usegerberextensions false)
+      (usegerberextensions true)
       (usegerberattributes true)
       (usegerberadvancedattributes true)
-      (creategerberjobfile true)
+      (creategerberjobfile false)
       (svguseinch false)
       (svgprecision 6)
@@
       (plotinvisibletext false)
       (sketchpadsonfab false)
-      (subtractmaskfromsilk false)
+      (subtractmaskfromsilk true)
       (outputformat 1)
       (mirror false)
-      (drillshape 1)
+      (drillshape 0)
       (scaleselection 1)
-      (outputdirectory "")
+      (outputdirectory "Gerbers")
     )
   )
@@
     (property "Sheetname" "")
     (attr smd)
-    (fp_text reference "F1" (at 2.82 0.08) (layer "F.SilkS")
+    (fp_text reference "F1" (at -2.66 0.08) (layer "F.SilkS")
       (effects (font (size 0.8 0.8) (thickness 0.1)))
     )
@@
     (property "Sheetname" "")
     (attr smd)
-    (fp_text reference "C4" (at 2.03 0.06) (layer "F.SilkS")
+    (fp_text reference "C4" (at 1.72 -0.04) (layer "F.SilkS")
       (effects (font (size 0.8 0.8) (thickness 0.1)))
     )
@@
     (property "uuid" "std:9dfaea9d47bf4a0f92de24ec40f7b62e")
     (attr through_hole)
-    (fp_text reference "U3" (at -4.553768 -4.36992) (layer "F.SilkS")
+    (fp_text reference "U3" (at -1.25865 -4.624478) (layer "F.SilkS")
       (effects (font (size 0.8 0.8) (thickness 0.1)) (justify left))
     )
@@
   )
   (footprint "LOGO" (layer "F.Cu")
-    (at 148.082 122.936)
+    (at 148.87 121.59)
     (attr board_only exclude_from_pos_files exclude_from_bom)
     (fp_text reference "" (at 0 0) (layer "F.SilkS")
@@
     (effects (font (size 0.8 0.8) (thickness 0.1)) (justify mirror))
   )
-  (gr_text "NRST" (at 167.32 106.69) (layer "B.SilkS")
+  (gr_text "NRST" (at 167.37 106.69) (layer "B.SilkS")
     (effects (font (size 0.8 0.8) (thickness 0.1)) (justify mirror))
   )
@@
     (effects (font (size 0.8 0.8) (thickness 0.1)) (justify mirror))
   )
+  (gr_text "PA13/SWDIO" (at 159.93 126.66 45) (layer "B.SilkS")
+    (effects (font (size 0.4 0.4) (thickness 0.1)) (justify mirror))
+  )
   (gr_text "PB8\n" (at 167.64 109.23) (layer "B.SilkS")
     (effects (font (size 0.8 0.8) (thickness 0.1)) (justify mirror))
@@
     (effects (font (size 1.5 1.5) (thickness 0.2)) (justify mirror))
   )
+  (gr_text "VDD_3.3V" (at 151.89 127.08 45) (layer "B.SilkS")
+    (effects (font (size 0.4 0.4) (thickness 0.1)) (justify mirror))
+  )
+  (gr_text "PA14/SWCLK" (at 154.82 126.63 45) (layer "B.SilkS")
+    (effects (font (size 0.4 0.4) (thickness 0.1)) (justify mirror))
+  )
   (gr_text "PB2" (at 167.64 124.47) (layer "B.SilkS")
     (effects (font (size 0.8 0.8) (thickness 0.1)) (justify mirror))
@@
     (effects (font (size 0.8 0.8) (thickness 0.1)) (justify mirror))
   )
+  (gr_text "GND" (at 156.51 127.61 45) (layer "B.SilkS")
+    (effects (font (size 0.4 0.4) (thickness 0.1)) (justify mirror))
+  )
   (gr_text "PA8" (at 142.27 116.85) (layer "B.SilkS")
     (effects (font (size 0.8 0.8) (thickness 0.1)) (justify mirror))
@@
     (effects (font (size 0.8 0.8) (thickness 0.1)) (justify mirror))
   )
-  (gr_text "5V" (at 168.07 96.55) (layer "B.SilkS")
+  (gr_text "5V" (at 168.19 96.55) (layer "B.SilkS")
     (effects (font (size 0.8 0.8) (thickness 0.1)) (justify mirror))
   )
@@
     (effects (font (size 0.8 0.8) (thickness 0.1)) (justify mirror))
   )
-  (gr_text "3.3V" (at 167.41 101.6) (layer "B.SilkS")
+  (gr_text "3.3V" (at 167.65 101.61) (layer "B.SilkS")
     (effects (font (size 0.8 0.8) (thickness 0.1)) (justify mirror))
   )
-  (gr_text "GND" (at 167.6 99.06) (layer "B.SilkS")
+  (gr_text "GND" (at 167.72 99.04) (layer "B.SilkS")
     (effects (font (size 0.8 0.8) (thickness 0.1)) (justify mirror))
   )
@@
     (effects (font (size 0.8 0.8) (thickness 0.1)))
   )
+  (gr_text "VDD_3.3V" (at 151.88 127.08 45) (layer "F.SilkS")
+    (effects (font (size 0.4 0.4) (thickness 0.1)))
+  )
   (gr_text "PA4" (at 142.24 106.68) (layer "F.SilkS")
     (effects (font (size 0.8 0.8) (thickness 0.1)))
   )
-  (gr_text "UINIO-EVB-STM32L051K8    Version 1.0.0" (at 154.94 126.746) (layer "F.SilkS")
-    (effects (font (size 0.5 0.5) (thickness 0.1)))
+  (gr_text "UINIO-EVB-STM32L051K8" (at 145.12 122.19 90) (layer "F.SilkS")
+    (effects (font (size 0.6 0.6) (thickness 0.15)))
+  )
+  (gr_text "GND" (at 156.51 127.62 45) (layer "F.SilkS")
+    (effects (font (size 0.4 0.4) (thickness 0.1)))
+  )
+  (gr_text "PA13/SWDIO" (at 159.93 126.68 45) (layer "F.SilkS")
+    (effects (font (size 0.4 0.4) (thickness 0.1)))
   )
   (gr_text "PA0" (at 142.24 96.52) (layer "F.SilkS")
@@
     (effects (font (size 0.8 0.8) (thickness 0.1)))
   )
-  (gr_text "NRST" (at 167.259 106.68) (layer "F.SilkS")
+  (gr_text "NRST" (at 167.309 106.68) (layer "F.SilkS")
     (effects (font (size 0.8 0.8) (thickness 0.1)))
   )
@@
     (effects (font (size 0.8 0.8) (thickness 0.1)))
   )
-  (gr_text "5V" (at 167.98 96.52) (layer "F.SilkS")
+  (gr_text "5V" (at 168.13 96.52) (layer "F.SilkS")
     (effects (font (size 0.8 0.8) (thickness 0.1)))
   )
+  (gr_text "Version 1.0.0" (at 148.81 125.04) (layer "F.SilkS")
+    (effects (font (size 0.4 0.4) (thickness 0.075)))
+  )
   (gr_text "系统复位" (at 164.48 109.38 90) (layer "F.SilkS")
     (effects (font (size 1 1) (thickness 0.15)))
@@
     (effects (font (size 0.8 0.8) (thickness 0.1)))
   )
-  (gr_text "3.3V" (at 167.386 101.6) (layer "F.SilkS")
+  (gr_text "3.3V" (at 167.61 101.61) (layer "F.SilkS")
     (effects (font (size 0.8 0.8) (thickness 0.1)))
   )
@@
     (effects (font (size 0.8 0.8) (thickness 0.1)))
   )
+  (gr_text "PA14/SWCLK" (at 154.81 126.64 45) (layer "F.SilkS")
+    (effects (font (size 0.4 0.4) (thickness 0.1)))
+  )
   (gr_text "PB3" (at 167.64 121.92) (layer "F.SilkS")
     (effects (font (size 0.8 0.8) (thickness 0.1)))
@@
     (effects (font (size 0.8 0.8) (thickness 0.1)))
   )
-  (gr_text "GND" (at 167.615031 99.050017) (layer "F.SilkS")
+  (gr_text "GND" (at 167.72 99.04) (layer "F.SilkS")
     (effects (font (size 0.8 0.8) (thickness 0.1)))
   )

Commit message: Re-layout and wiring
Parts:
- R1: value 10K -> 1K
- R2: value R -> 10K
- R3: value 1K -> R
- USB1: value USB_Type_C_16Pin -> USB_Type_C_6Pin; footprint Uinio:USB-C-SMD_TYPEC-304J-BCP16 -> Uinio:USB-TYPEC-250-BRP6L68
- moved ? 36.4 mm to (156.7, 86.0)
- moved R1 26.4 mm to (165.5, 87.5), turned to 180 degrees
- moved C10 17.8 mm to (160.5, 106.8), turned to 0 degrees
- moved C11 16.6 mm to (158.7, 106.8)
- moved C3 16.3 mm to (156.5, 95.8), turned to 180 degrees
- moved Y1 13.9 mm to (159.6, 109.5), turned to -90 degrees
- moved R2 13.2 mm to (155.5, 96.2)
- moved U2 12.7 mm to (156.6, 99.3)
- moved USB1 12.2 mm to (156.6, 87.9)
- moved D1 11.6 mm to (165.5, 89.5)
- moved C2 11.4 mm to (149.2, 91.3)
- moved U1 11.2 mm to (148.8, 88.8)
- moved F1 11.2 mm to (163.2, 89.3), turned to -90 degrees
- moved C1 10.9 mm to (149.2, 86.4)
- moved SW1 10.9 mm to (153.2, 99.8)
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Connections:
- J1 pad 12: /PA11/USB_Data_N -> /PA11
- J1 pad 13: /PA12/USB_Data_P -> /PA12
- R1 pad 1: GND -> Net-(D1-Pad2)
- R1 pad 2: /BOOT0 -> /VDD_5V
- R2 pad 1: /VDD_3.3V -> GND
- R2 pad 2: /NRST -> /BOOT0
- R3 pad 1: Net-(D1-Pad2) -> /VDD_3.3V
- R3 pad 2: /VDD_5V -> /NRST
- U3 pad 21: /PA11/USB_Data_N -> /PA11
- U3 pad 22: /PA12/USB_Data_P -> /PA12
Routing:
- net GND: track 124.1 -> 178.7 mm, vias 10 -> 13
- net /PA12/USB_Data_P: track 46.2 -> 0.00 mm, vias 4 -> 0
- net /PA11/USB_Data_N: track 43.4 -> 0.00 mm, vias 4 -> 0
- net /PA7/MOSI: track 50.4 -> 21.9 mm, vias 2 -> 0
- net /PB4: track 32.5 -> 8.50 mm
- net /PB5: track 33.8 -> 9.97 mm
- net /PB6: track 35.2 -> 11.5 mm
- net /PB7: track 36.5 -> 13.3 mm
- net /PB3: track 31.1 -> 8.23 mm
- net /PB8: track 36.7 -> 14.3 mm
- net /PA5/SCLK: track 37.7 -> 21.5 mm, vias 1 -> 0
- net /PA2: track 34.6 -> 19.7 mm, vias 2 -> 0
- net /PA1: track 35.3 -> 23.2 mm, vias 2 -> 0
- net /PA13/SWDIO: track 25.4 -> 13.6 mm, vias 0 -> 1
- net /NRST: track 37.2 -> 27.2 mm
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Other:
- board size 34.4 x 36.6 mm -> 21.2 x 48.4 mm
