File: UINIO-MCU-STM32L051K8.kicad_pcb (KiCad board)
At the start: 2 copper layers, 48.4 x 21.2 mm, 31 parts, among them J1 Conn_01x14_Male, J2 Conn_01x14_Male, J3 Conn_01x04_Male, SW1 SW_Push, SW2 SW_Push, U1 ME6211C33M5G-N, U2 W25Q128JVSSIQ, U3 STM32L051K8U6, Y1 Crystal_GND24

Commit message: Release UINIO-MCU-STM32L051K8 1.0.0.
Routing:
- net GND: track 180.4 -> 192.4 mm, vias 12 -> 20
- net Net-(F1-Pad1): track 13.5 -> 14.3 mm

Commit message: Update PCB layout.
Parts:
- added ?: , LOGO, F.Cu at (137.9, 99.9)
- C10, C11: value 8pF -> 22pF
- Y1: value Crystal_GND24 -> 12MHz
- moved J3 7.62 mm to (130.4, 96.0), turned to 0 degrees
- moved C8 0.25 mm to (149.2, 99.0)
- moved C6 0.12 mm to (149.2, 100.4)
Routing:
- net GND: track 192.4 -> 182.9 mm, vias 20 -> 23
- net /VDD_3.3V: track 104.7 -> 109.6 mm, vias 5 -> 8
- net /PA13/SWDIO: track 13.6 -> 11.8 mm
- net /PA15: track 13.4 -> 15.1 mm
- net /PA14/SWCLK: track 10.6 -> 11.6 mm

Commit message: Update PCB board.
Parts:
- removed HOLE1, HOLE2, HOLE3, HOLE4: Hole-1mm, Uinio:Hole-1mm
- C10, C11: value 22pF -> 6pF
- Y1: value 12MHz -> FC135-32.768; footprint Crystal:Crystal_SMD_3225-4Pin_3.2x2.5mm -> Uinio:CRYSTAL-FC135-32.768
- moved C11 1.28 mm to (151.1, 102.2)
- moved C10 1.27 mm to (151.1, 104.0)
- moved Y1 0.53 mm to (149.1, 103.1), turned to -90 degrees
Connections:
- Y1 pad 2: GND -> Net-(C10-Pad2)
Routing:
- net Net-(C11-Pad2): track 11.5 -> 7.23 mm, vias 2 -> 0
- net GND: track 182.9 -> 180.2 mm
- net Net-(C10-Pad2): track 8.84 -> 7.63 mm

Commit message: Update PCB Layout.
Parts:
- added Hole1: Hole-1mm, Uinio:Hole-1mm, F.Cu at (130.5, 91.8)
- added Hole2: Hole-1mm, Uinio:Hole-1mm, F.Cu at (130.6, 107.6)
- added Hole3: Hole-1mm, Uinio:Hole-1mm, F.Cu at (175.0, 107.6)
- added Hole4: Hole-1mm, Uinio:Hole-1mm, F.Cu at (174.9, 91.8)
- moved ? 0.33 mm to (137.6, 99.9)
- moved J3 0.30 mm to (130.1, 96.0)
- moved J2 0.11 mm to (166.0, 108.5)
Routing:
- net GND: track 180.2 -> 177.0 mm, vias 23 -> 24
Other:
- board size 48.4 x 21.2 mm -> 48.4 x 20.5 mm
