File: UINIO-MCU-STM32L051K8.kicad_pcb (KiCad board)
At the start: 2 copper layers, 48.4 x 20.5 mm, 33 parts, among them J1 Conn_01x14_Male, J2 Conn_01x14_Male, J3 Conn_01x04_Male, SW1 SW_Push, SW2 SW_Push, U1 ME6211, U2 W25Q128JVSSIQ, U3 STM32L051K8U6, Y1 FC135-32.768

Commit message: Update folders.
Parts:
- C1, C2: value CAP_0402 -> 1uF
- C10, C11: value C -> 6pF
- C3, C4, C5, C6, C7, C9: value C -> 0.1uF
- C8: value C -> 1uF
- D1: value LED -> Red LED
- R1: value R -> 1K
- R2, R3: value R -> 10K
Other:
- board text added: "Version 3.1.0"
- board text removed: "Version 3.0.0"
Changed lines of the file:
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@@
   (title_block
     (title "UINIO-MCU-STM32L051K8")
-    (date "2023-01-11")
-    (rev "Version 3.0.0")
+    (date "2023-01-24")
+    (rev "Version 3.1.0")
     (company "电子技术博客 UinIO.com")
   )
@@
       (effects (font (size 0.6 0.6) (thickness 0.1)))
     )
-    (fp_text value "R" (at 0 1.17) (layer "F.Fab")
+    (fp_text value "10K" (at 0 1.17) (layer "F.Fab")
       (effects (font (size 1 1) (thickness 0.15)))
     )
@@
       (effects (font (size 0.6 0.6) (thickness 0.1)))
     )
-    (fp_text value "C" (at 0 1.16) (layer "F.Fab")
+    (fp_text value "0.1uF" (at 0 1.16) (layer "F.Fab")
       (effects (font (size 1 1) (thickness 0.15)))
     )
@@
       (effects (font (size 0.6 0.6) (thickness 0.1)))
     )
-    (fp_text value "C" (at 0 1.16) (layer "F.Fab")
+    (fp_text value "0.1uF" (at 0 1.16) (layer "F.Fab")
       (effects (font (size 1 1) (thickness 0.15)))
     )
@@
       (effects (font (size 0.6 0.6) (thickness 0.1)))
     )
-    (fp_text value "R" (at 0 1.17 90) (layer "F.Fab")
+    (fp_text value "1K" (at 0 1.17 90) (layer "F.Fab")
       (effects (font (size 1 1) (thickness 0.15)))
     )
@@
       (effects (font (size 0.6 0.6) (thickness 0.1)))
     )
-    (fp_text value "C" (at 0 1.16) (layer "F.Fab")
+    (fp_text value "1uF" (at 0 1.16) (layer "F.Fab")
       (effects (font (size 1 1) (thickness 0.15)))
     )
@@
       (effects (font (size 0.6 0.6) (thickness 0.1)))
     )
-    (fp_text value "C" (at 0 1.16) (layer "F.Fab")
+    (fp_text value "0.1uF" (at 0 1.16) (layer "F.Fab")
       (effects (font (size 1 1) (thickness 0.15)))
     )
@@
       (effects (font (size 0.6 0.6) (thickness 0.1)))
     )
-    (fp_text value "C" (at 0 1.16) (layer "F.Fab")
+    (fp_text value "0.1uF" (at 0 1.16) (layer "F.Fab")
       (effects (font (size 1 1) (thickness 0.15)))
     )
@@
       (effects (font (size 0.6 0.6) (thickness 0.1)))
     )
-    (fp_text value "R" (at 0 1.17) (layer "F.Fab")
+    (fp_text value "10K" (at 0 1.17) (layer "F.Fab")
       (effects (font (size 1 1) (thickness 0.15)))
     )
@@
       (effects (font (size 0.6 0.6) (thickness 0.1)))
     )
-    (fp_text value "LED" (at 0 1.43) (layer "F.Fab")
+    (fp_text value "Red LED" (at 0 1.43) (layer "F.Fab")
       (effects (font (size 1 1) (thickness 0.15)))
     )
@@
       (effects (font (size 1.524 1.524) (thickness 0.254)) (justify left bottom))
     )
-    (fp_text value "CAP_0402" (at 0.6477 -2.7305 -270 unlocked) (layer "F.SilkS") hide
+    (fp_text value "1uF" (at 0.6477 -2.7305 -270 unlocked) (layer "F.SilkS") hide
       (effects (font (size 1.524 1.524) (thickness 0.254)) (justify left bottom))
     )
@@
       (effects (font (size 0.6 0.6) (thickness 0.1)))
     )
-    (fp_text value "C" (at 0 1.16) (layer "F.Fab")
+    (fp_text value "0.1uF" (at 0 1.16) (layer "F.Fab")
       (effects (font (size 1 1) (thickness 0.15)))
     )
@@
       (effects (font (size 0.6 0.6) (thickness 0.1)))
     )
-    (fp_text value "C" (at 0 1.16 90) (layer "F.Fab")
+    (fp_text value "6pF" (at 0 1.16 90) (layer "F.Fab")
       (effects (font (size 1 1) (thickness 0.15)))
     )
@@
       (effects (font (size 0.6 0.6) (thickness 0.1)))
     )
-    (fp_text value "C" (at 0 1.16 90) (layer "F.Fab")
+    (fp_text value "6pF" (at 0 1.16 90) (layer "F.Fab")
       (effects (font (size 1 1) (thickness 0.15)))
     )
@@
       (effects (font (size 1.524 1.524) (thickness 0.254)) (justify left bottom))
     )
-    (fp_text value "CAP_0402" (at 0.6477 -2.7305 -270 unlocked) (layer "F.SilkS") hide
+    (fp_text value "1uF" (at 0.6477 -2.7305 -270 unlocked) (layer "F.SilkS") hide
       (effects (font (size 1.524 1.524) (thickness 0.254)) (justify left bottom))
     )
@@
       (effects (font (size 0.6 0.6) (thickness 0.1)) (justify mirror))
     )
-    (fp_text value "C" (at 0 -1.16 90) (layer "B.Fab")
+    (fp_text value "0.1uF" (at 0 -1.16 90) (layer "B.Fab")
       (effects (font (size 1 1) (thickness 0.15)) (justify mirror))
     )
@@
     (effects (font (size 0.7 0.7) (thickness 0.1)) (justify mirror))
   )
-  (gr_text "Version 3.0.0" (at 171.27 99.71 -90) (layer "B.SilkS")
+  (gr_text "Version 3.1.0" (at 171.27 99.71 -90) (layer "B.SilkS")
     (effects (font (size 0.7 0.7) (thickness 0.1)) (justify mirror))
   )
@@
   )
   (gr_text "STM32L051K8U6" (at 150.18 96.42) (layer "F.SilkS")
-    (effects (font (size 0.7 0.7) (thickness 0.16)))
+    (effects (font (size 0.8 0.8) (thickness 0.2)))
   )
   (gr_text "5V" (at 165.955 106.414 270) (layer "F.SilkS")

Commit message: Release UINIO-MCU-STM32L051K8 version 3.1.0.
Parts:
- Y1: value FC135-32.768 -> Crystal-FC135-32.768
Routing:
- net GND: track 180.8 -> 185.6 mm, vias 24 -> 25

Commit message: Release UINIO-MCU-STM32L051K8 version 3.1.0.
Routing:
- net GND: track 185.6 -> 186.5 mm
Changed lines of the file:
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@@
     (property "uuid" "std:2c2510636cee4069ad38e03b5f14209b")
     (attr through_hole)
-    (fp_text reference "USB1" (at 1.13 1.42 270) (layer "F.SilkS")
+    (fp_text reference "USB1" (at -1.3 1.06 90) (layer "F.SilkS")
       (effects (font (size 0.6 0.6) (thickness 0.1)) (justify left))
     )
@@
     (property "Sheetname" "")
     (attr smd)
-    (fp_text reference "D1" (at -1.945 0.04 90) (layer "F.SilkS")
+    (fp_text reference "D1" (at -1.955 0.04 90) (layer "F.SilkS")
       (effects (font (size 0.6 0.6) (thickness 0.1)))
     )
@@
     (property "Sheetname" "")
     (attr through_hole)
-    (fp_text reference "U1" (at 0 0.876 90) (layer "F.SilkS")
+    (fp_text reference "U1" (at 0.03 0.59 90) (layer "F.SilkS")
       (effects (font (size 0.6 0.6) (thickness 0.1)) (justify left))
     )
@@
   (segment (start 156.78 99.73) (end 156.75 99.76) (width 0.3) (layer "F.Cu") (net 1))
   (segment (start 173.09 91.88) (end 172 91.88) (width 0.3) (layer "F.Cu") (net 1))
-  (segment (start 168.85 108.62) (end 169.4575 108.62) (width 0.5) (layer "F.Cu") (net 1))
   (segment (start 168.3 91.88) (end 168.3 90.53) (width 0.3) (layer "F.Cu") (net 1))
   (segment (start 149.64 98.06) (end 149.64 99.01) (width 0.3) (layer "F.Cu") (net 1))
@@
   (segment (start 144.85 105.93) (end 143.287147 104.367147) (width 0.3) (layer "F.Cu") (net 1))
   (segment (start 172.59 90.05) (end 173.08 90.54) (width 0.3) (layer "F.Cu") (net 1))
+  (segment (start 167.82 108.62) (end 169.4575 108.62) (width 0.5) (layer "F.Cu") (net 1))
   (segment (start 163.52 101.87) (end 163.53 101.88) (width 0.5) (layer "F.Cu") (net 1))
   (segment (start 171.26 95.41) (end 171.26 95.98) (width 0.5) (layer "F.Cu") (net 1))
@@
   (segment (start 148.22 101.06) (end 150.51 101.06) (width 0.2) (layer "F.Cu") (net 1))
   (segment (start 163.5 99.68) (end 161.93 99.68) (width 0.3) (layer "F.Cu") (net 1))
-  (segment (start 168.26 108.03) (end 168.85 108.62) (width 0.5) (layer "F.Cu") (net 1))
   (segment (start 151.95 104.51) (end 151.14 104.51) (width 0.3) (layer "F.Cu") (net 1))
   (segment (start 171.26 104.05) (end 171.26 103.48) (width 0.5) (layer "F.Cu") (net 1))
@@
   (via (at 139.42 93.73) (size 0.5) (drill 0.3) (layers "F.Cu" "B.Cu") (free) (net 1))
   (via (at 163.52 101.87) (size 0.7) (drill 0.3) (layers "F.Cu" "B.Cu") (net 1))
-  (via (at 168.26 108.03) (size 0.9) (drill 0.5) (layers "F.Cu" "B.Cu") (net 1))
+  (via (at 167.82 108.62) (size 0.9) (drill 0.5) (layers "F.Cu" "B.Cu") (net 1))
   (via (at 144.24 99.17) (size 0.5) (drill 0.2) (layers "F.Cu" "B.Cu") (remove_unused_layers) (net 1))
   (via (at 141.92 106.8) (size 0.5) (drill 0.3) (layers "F.Cu" "B.Cu") (free) (net 1))
@@
   (segment (start 152.53 94.27) (end 152.53 95.93) (width 0.3) (layer "B.Cu") (net 1))
   (segment (start 145 105.96) (end 158.08 105.96) (width 0.3) (layer "B.Cu") (net 1))
-  (segment (start 171.26 105.05) (end 171.26 104.05) (width 0.5) (layer "B.Cu") (net 1))
-  (segment (start 168.28 108.03) (end 171.26 105.05) (width 0.5) (layer "B.Cu") (net 1))
+  (segment (start 171.26 105.18) (end 171.26 104.05) (width 0.5) (layer "B.Cu") (net 1))
   (segment (start 151.84 93.58) (end 152.53 94.27) (width 0.3) (layer "B.Cu") (net 1))
   (segment (start 145.14 93.58) (end 151.84 93.58) (width 0.3) (layer "B.Cu") (net 1))
@@
   (segment (start 145.12 93.6) (end 145.14 93.58) (width 0.3) (layer "B.Cu") (net 1))
   (segment (start 139.88 105.99) (end 144.91 105.99) (width 0.3) (layer "B.Cu") (net 1))
+  (segment (start 167.82 108.62) (end 171.26 105.18) (width 0.5) (layer "B.Cu") (net 1))
   (segment (start 163.56 106.7) (end 163.56 108.38) (width 0.5) (layer "B.Cu") (net 1))
   (segment (start 169.19 95.41) (end 171.26 95.41) (width 0.5) (layer "B.Cu") (net 1))
@@
   (segment (start 163.44 108.26) (end 163.44 107.11) (width 0.3) (layer "B.Cu") (net 1))
   (segment (start 166.89 93.37) (end 168.955 95.435) (width 0.3) (layer "B.Cu") (net 1))
-  (segment (start 168.26 108.03) (end 168.28 108.03) (width 0.5) (layer "B.Cu") (net 1))
   (segment (start 158.405 103.21) (end 158.405 104.715) (width 0.3) (layer "B.Cu") (net 1))
   (segment (start 144.97 105.93) (end 145 105.96) (width 0.3) (layer "B.Cu") (net 1))

Commit message: Release UINIO-MCU-STM32L051K8 version 3.1.0.
Parts:
- C1, C2: footprint Uinio:CAP_0402 -> Capacitor_SMD:C_0402_1005Metric
Changed lines of the file:
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@@
       ) (layer "F.SilkS") (width 0) (fill solid))
   )
-  (footprint "Uinio:CAP_0402" (layer "F.Cu")
+  (footprint "Capacitor_SMD:C_0402_1005Metric" (layer "F.Cu")
     (at 168.3 92.36 -90)
+    (descr "Capacitor SMD 0402 (1005 Metric), square (rectangular) end terminal, IPC_7351 nominal, (Body size source: IPC-SM-782 page 76, https://www.pcb-3d.com/wordpress/wp-content/uploads/ipc-sm-782a_amendment_1_and_2.pdf), generated with kicad-footprint-generator")
+    (tags "capacitor")
     (property "ALTIUM_VALUE" "0.1u")
     (property "BOM名称" "无极性贴片电容")
@@
     (property "Sheetname" "")
     (property "材质" "X7R")
-    (fp_text reference "C2" (at 0.6604 1.2192 -270 unlocked) (layer "F.SilkS") hide
-      (effects (font (size 1.524 1.524) (thickness 0.254)) (justify left bottom))
+    (attr smd)
+    (fp_text reference "C2" (at -1.58 0 -90) (layer "F.SilkS")
+      (effects (font (size 0.6 0.6) (thickness 0.1)))
     )
-    (fp_text value "1uF" (at 0.6477 -2.7305 -270 unlocked) (layer "F.SilkS") hide
-      (effects (font (size 1.524 1.524) (thickness 0.254)) (justify left bottom))
+    (fp_text value "1uF" (at 0 1.16 -90) (layer "F.Fab")
+      (effects (font (size 1 1) (thickness 0.15)))
     )
-    (fp_line (start -0.0762 0.2286) (end -0.1651 0.2286) (layer "F.SilkS") (width 0.0254))
-    (fp_line (start 0.0762 -0.2286) (end 0.0762 0.2286) (layer "F.SilkS") (width 0.0254))
-    (fp_line (start 0.1651 -0.2286) (end 0.1651 0.2286) (layer "F.SilkS") (width 0.0254))
-    (fp_line (start -0.1651 -0.2286) (end -0.1651 0.2286) (layer "F.SilkS") (width 0.0254))
-    (fp_line (start 0.1651 -0.2286) (end 0.0762 -0.2286) (layer "F.SilkS") (width 0.0254))
-    (fp_line (start -0.0762 -0.2286) (end -0.1651 -0.2286) (layer "F.SilkS") (width 0.0254))
-    (fp_line (start 0.1651 0.2286) (end 0.0762 0.2286) (layer "F.SilkS") (width 0.0254))
-    (fp_line (start -0.0762 -0.2286) (end -0.0762 0.2286) (layer "F.SilkS") (width 0.0254))
-    (fp_line (start -0.889 -0.4318) (end -0.889 0.4318) (layer "Eco1.User") (width 0.0508))
-    (fp_line (start 0.889 -0.4318) (end -0.889 -0.4318) (layer "Eco1.User") (width 0.0508))
-    (fp_line (start 0.889 -0.4318) (end 0.889 0.4318) (layer "Eco1.User") (width 0.0508))
-    (fp_line (start 0.889 0.4318) (end -0.889 0.4318) (layer "Eco1.User") (width 0.0508))
-    (fp_line (start 0.499999 0.250013) (end -0.500001 0.250013) (layer "B.Fab") (width 0.0508))
-    (fp_line (start 0.499999 -0.250002) (end -0.500001 -0.250002) (layer "B.Fab") (width 0.0508))
-    (fp_line (start -0.500001 -0.250002) (end -0.500001 0.250013) (layer "B.Fab") (width 0.0508))
-    (fp_line (start 0.152482 -0.000081) (end -0.152318 -0.000081) (layer "B.Fab") (width 0.0508))
-    (fp_line (start 0.499999 -0.250012) (end 0.499999 0.250013) (layer "B.Fab") (width 0.0508))
-    (fp_line (start 0 -0.1524) (end 0 0.1524) (layer "B.Fab") (width 0.0508))
-    (pad "1" smd roundrect (at -0.508 0) (size 0.508 0.508) (layers "F.Cu" "F.Paste" "F.Mask") (roundrect_rratio 0.25)
+    (fp_text user "${REFERENCE}" (at 0 0 -90) (layer "F.Fab")
+      (effects (font (size 0.25 0.25) (thickness 0.04)))
+    )
+    (fp_line (start -0.107836 -0.36) (end 0.107836 -0.36) (layer "F.SilkS") (width 0.12))
+    (fp_line (start -0.107836 0.36) (end 0.107836 0.36) (layer "F.SilkS") (width 0.12))
+    (fp_line (start -0.91 -0.46) (end 0.91 -0.46) (layer "F.CrtYd") (width 0.05))
+    (fp_line (start -0.91 0.46) (end -0.91 -0.46) (layer "F.CrtYd") (width 0.05))
+    (fp_line (start 0.91 -0.46) (end 0.91 0.46) (layer "F.CrtYd") (width 0.05))
+    (fp_line (start 0.91 0.46) (end -0.91 0.46) (layer "F.CrtYd") (width 0.05))
+    (fp_line (start -0.5 0.25) (end -0.5 -0.25) (layer "F.Fab") (width 0.1))
+    (fp_line (start -0.5 -0.25) (end 0.5 -0.25) (layer "F.Fab") (width 0.1))
+    (fp_line (start 0.5 -0.25) (end 0.5 0.25) (layer "F.Fab") (width 0.1))
+    (fp_line (start 0.5 0.25) (end -0.5 0.25) (layer "F.Fab") (width 0.1))
+    (pad "1" smd roundrect (at -0.48 0 270) (size 0.56 0.62) (layers "F.Cu" "F.Paste" "F.Mask") (roundrect_rratio 0.25)
       (net 1 "GND") (pinfunction "1") (pintype "passive"))
-    (pad "2" smd roundrect (at 0.508 0) (size 0.508 0.508) (layers "F.Cu" "F.Paste" "F.Mask") (roundrect_rratio 0.25)
+    (pad "2" smd roundrect (at 0.48 0 270) (size 0.56 0.62) (layers "F.Cu" "F.Paste" "F.Mask") (roundrect_rratio 0.25)
       (net 3 "/VDD_3.3V") (pinfunction "2") (pintype "passive"))
-    (model "${KIPRJMOD}/ALTIUM_EMBEDDED_MODELS/CAPC1005X05L.step"
-      (offset (xyz 0.000082 0.000081 0))
+    (model "${KICAD6_3DMODEL_DIR}/Capacitor_SMD.3dshapes/C_0402_1005Metric.wrl"
+      (offset (xyz 0 0 0))
       (scale (xyz 1 1 1))
-      (rotate (xyz -0 -0 0))
+      (rotate (xyz 0 0 0))
     )
   )
@@
     )
   )
-  (footprint "Uinio:CAP_0402" (layer "F.Cu")
+  (footprint "Capacitor_SMD:C_0402_1005Metric" (layer "F.Cu")
     (at 173.09 92.36 -90)
+    (descr "Capacitor SMD 0402 (1005 Metric), square (rectangular) end terminal, IPC_7351 nominal, (Body size source: IPC-SM-782 page 76, https://www.pcb-3d.com/wordpress/wp-content/uploads/ipc-sm-782a_amendment_1_and_2.pdf), generated with kicad-footprint-generator")
+    (tags "capacitor")
     (property "ALTIUM_VALUE" "0.1u")
     (property "BOM名称" "无极性贴片电容")
@@
     (property "Sheetname" "")
     (property "材质" "X7R")
-    (fp_text reference "C1" (at 0.6604 1.2192 -270 unlocked) (layer "F.SilkS") hide
-      (effects (font (size 1.524 1.524) (thickness 0.254)) (justify left bottom))
+    (attr smd)
+    (fp_text reference "C1" (at -1.58 0.02 -90) (layer "F.SilkS")
+      (effects (font (size 0.6 0.6) (thickness 0.1)))
     )
-    (fp_text value "1uF" (at 0.6477 -2.7305 -270 unlocked) (layer "F.SilkS") hide
-      (effects (font (size 1.524 1.524) (thickness 0.254)) (justify left bottom))
+    (fp_text value "1uF" (at 0 1.16 -90) (layer "F.Fab")
+      (effects (font (size 1 1) (thickness 0.15)))
     )
-    (fp_line (start 0.0762 -0.2286) (end 0.0762 0.2286) (layer "F.SilkS") (width 0.0254))
-    (fp_line (start -0.0762 0.2286) (end -0.1651 0.2286) (layer "F.SilkS") (width 0.0254))
-    (fp_line (start 0.1651 -0.2286) (end 0.0762 -0.2286) (layer "F.SilkS") (width 0.0254))
-    (fp_line (start -0.0762 -0.2286) (end -0.1651 -0.2286) (layer "F.SilkS") (width 0.0254))
-    (fp_line (start 0.1651 0.2286) (end 0.0762 0.2286) (layer "F.SilkS") (width 0.0254))
-    (fp_line (start -0.0762 -0.2286) (end -0.0762 0.2286) (layer "F.SilkS") (width 0.0254))
-    (fp_line (start 0.1651 -0.2286) (end 0.1651 0.2286) (layer "F.SilkS") (width 0.0254))
-    (fp_line (start -0.1651 -0.2286) (end -0.1651 0.2286) (layer "F.SilkS") (width 0.0254))
-    (fp_line (start 0.889 0.4318) (end -0.889 0.4318) (layer "Eco1.User") (width 0.0508))
-    (fp_line (start -0.889 -0.4318) (end -0.889 0.4318) (layer "Eco1.User") (width 0.0508))
-    (fp_line (start 0.889 -0.4318) (end -0.889 -0.4318) (layer "Eco1.User") (width 0.0508))
-    (fp_line (start 0.889 -0.4318) (end 0.889 0.4318) (layer "Eco1.User") (width 0.0508))
-    (fp_line (start 0.499999 -0.250012) (end 0.499999 0.250013) (layer "B.Fab") (width 0.0508))
-    (fp_line (start 0.499999 -0.250002) (end -0.500001 -0.250002) (layer "B.Fab") (width 0.0508))
-    (fp_line (start 0.152482 -0.000081) (end -0.152318 -0.000081) (layer "B.Fab") (width 0.0508))
-    (fp_line (start -0.500001 -0.250002) (end -0.500001 0.250013) (layer "B.Fab") (width 0.0508))
-    (fp_line (start 0 -0.1524) (end 0 0.1524) (layer "B.Fab") (width 0.0508))
-    (fp_line (start 0.499999 0.250013) (end -0.500001 0.250013) (layer "B.Fab") (width 0.0508))
-    (pad "1" smd roundrect (at -0.508 0) (size 0.508 0.508) (layers "F.Cu" "F.Paste" "F.Mask") (roundrect_rratio 0.25)
+    (fp_text user "${REFERENCE}" (at 0 0 -90) (layer "F.Fab")
+      (effects (font (size 0.25 0.25) (thickness 0.04)))
+    )
+    (fp_line (start -0.107836 0.36) (end 0.107836 0.36) (layer "F.SilkS") (width 0.12))
+    (fp_line (start -0.107836 -0.36) (end 0.107836 -0.36) (layer "F.SilkS") (width 0.12))
+    (fp_line (start -0.91 -0.46) (end 0.91 -0.46) (layer "F.CrtYd") (width 0.05))
+    (fp_line (start 0.91 0.46) (end -0.91 0.46) (layer "F.CrtYd") (width 0.05))
+    (fp_line (start 0.91 -0.46) (end 0.91 0.46) (layer "F.CrtYd") (width 0.05))
+    (fp_line (start -0.91 0.46) (end -0.91 -0.46) (layer "F.CrtYd") (width 0.05))
+    (fp_line (start 0.5 -0.25) (end 0.5 0.25) (layer "F.Fab") (width 0.1))
+    (fp_line (start 0.5 0.25) (end -0.5 0.25) (layer "F.Fab") (width 0.1))
+    (fp_line (start -0.5 0.25) (end -0.5 -0.25) (layer "F.Fab") (width 0.1))
+    (fp_line (start -0.5 -0.25) (end 0.5 -0.25) (layer "F.Fab") (width 0.1))
+    (pad "1" smd roundrect (at -0.48 0 270) (size 0.56 0.62) (layers "F.Cu" "F.Paste" "F.Mask") (roundrect_rratio 0.25)
       (net 1 "GND") (pinfunction "1") (pintype "passive"))
-    (pad "2" smd roundrect (at 0.508 0) (size 0.508 0.508) (layers "F.Cu" "F.Paste" "F.Mask") (roundrect_rratio 0.25)
+    (pad "2" smd roundrect (at 0.48 0 270) (size 0.56 0.62) (layers "F.Cu" "F.Paste" "F.Mask") (roundrect_rratio 0.25)
       (net 2 "/VDD_5V") (pinfunction "2") (pintype "passive"))
-    (model "${KIPRJMOD}/ALTIUM_EMBEDDED_MODELS/CAPC1005X05L.step"
-      (offset (xyz 0.000082 0.000081 0))
+    (model "${KICAD6_3DMODEL_DIR}/Capacitor_SMD.3dshapes/C_0402_1005Metric.wrl"
+      (offset (xyz 0 0 0))
       (scale (xyz 1 1 1))
-      (rotate (xyz -0 -0 0))
+      (rotate (xyz 0 0 0))
     )
   )

Commit message: Release UINIO-MCU-STM32L051K8 version 3.2.0.
Parts:
- moved Hole4 51.5 mm to (127.5, 111.7), turned to 180 degrees
- moved Hole3 48.9 mm to (127.5, 95.8), turned to 180 degrees
- moved C1 47.5 mm to (129.5, 111.1), turned to 90 degrees
- moved Hole1 46.0 mm to (172.1, 111.7), turned to 180 degrees
- moved R1 44.0 mm to (130.4, 94.9)
- moved J3 43.9 mm to (172.5, 107.5), turned to 180 degrees
- moved U1 43.5 mm to (131.9, 111.6), turned to 180 degrees
- moved Hole2 43.1 mm to (172.0, 95.9), turned to 180 degrees
- moved USB1 42.9 mm to (129.9, 103.8), turned to -90 degrees
- moved D1 40.3 mm to (132.3, 94.9), turned to 180 degrees
- moved F1 39.3 mm to (132.2, 97.1), turned to 0 degrees
- moved C2 38.8 mm to (134.3, 111.1), turned to 90 degrees
- moved J1 36.5 mm to (136.6, 112.5), turned to -90 degrees
- moved J2 32.3 mm to (136.6, 95.0), turned to -90 degrees
- moved ? 32.0 mm to (135.4, 103.7), turned to -90 degrees
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Connections:
- R1 pad 2: /VDD_5V -> /VDD_3.3V
Routing:
- net /VDD_3.3V: track 104.8 -> 126.1 mm, vias 5 -> 7
- net /VDD_5V: track 31.5 -> 28.0 mm
- net GND: track 186.5 -> 188.0 mm
- net /PA15: track 19.1 -> 20.3 mm
Other:
- outline, holes or cut-outs redrawn
- board text added: "Version 3.2.0"
- board text removed: "Version 3.1.0"

Commit message: Update version.
Parts:
- J1, J2: value Conn_01x14_Male -> Conn_01x14_Pin
- J3: value Conn_01x04_Male -> Conn_01x04_Pin

Commit message: Update PCB.
Parts:
- removed the ? at (164.9, 103.5)
- moved U2 0.09 mm to (142.3, 103.7)
- moved J1 0.06 mm to (136.6, 112.6)
- moved C4 0.05 mm to (158.8, 108.3)
Routing:
- net /PA6/MISO: track 31.8 -> 29.5 mm, vias 0 -> 2
- net Net-(F1-Pad1): track 15.2 -> 13.0 mm
- net /VDD_5V: track 28.0 -> 26.2 mm
- net /PA4/CS: track 36.1 -> 36.9 mm
- net /PA5/SCLK: track 21.4 -> 22.1 mm
- net /PA8: track 7.86 -> 7.20 mm
Other:
- board size 48.4 x 20.5 mm -> 48.3 x 20.3 mm
- board text added: "ARM"
- board text added: "STM32L051 K8U6"
- board text added: "UinIO.com"
- board text added: "Version 3.3.0"
- board text removed: "STM32L051K8U6"
- board text removed: "Version 3.2.0"
