File: UINIO-MCU-STM32L051K8.kicad_sch (KiCad schematic)
At the start: 26 parts, among them J1 Conn_01x14_Male, J2 Conn_01x14_Male, J3 Conn_01x04_Male, SW1 SW_Push, SW2 SW_Push, U1 ME6211C33M5G-N, U2 W25Q128JVSSIQ, U3 STM32L051K8U6, Y1 FC135-32.768

Commit message: Release UINIO-MCU-STM32L051K8 version 3.0.0.
Parts:
- C1, C2: value 1uF -> CAP_0402; footprint Capacitor_SMD:C_0402_1005Metric -> Uinio:CAP_0402
- C10, C11: value 6pF -> C
- C3, C4, C5, C7, C8, C9: value 0.1uF -> C
- C6: value 1uF -> C
- R1: value 1K -> R
- R2, R3: value 10K -> R
- U1: value ME6211C33M5G-N -> ME6211
Other:
- company: UinIO.com -> 电子技术博客 UinIO.com
Changed lines of the file:
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@@
   (title_block
     (title "UINIO-MCU-STM32L051K8")
-    (date "2022-09-29")
-    (rev "Hank")
-    (company "UinIO.com")
+    (date "2023-01-11")
+    (rev "Version 3.0.0")
+    (company "电子技术博客 UinIO.com")
   )
   (junction (at 35.56 99.06) (diameter 0) (color 0 0 0 0)
@@
     (in_bom yes) (on_board yes)
     (property "Reference" "C7" (id 0) (at 232.156 52.324 90))
-    (property "Value" "0.1uF" (id 1) (at 230.886 49.276 90))
+    (property "Value" "C" (id 1) (at 230.886 49.276 90))
     (property "Footprint" "Capacitor_SMD:C_0402_1005Metric" (id 2) (at 231.14 49.8348 0)
       (effects (font (size 1.27 1.27)) hide)
@@
     (in_bom yes) (on_board yes)
     (property "Reference" "C10" (id 0) (at 261.874 64.008 90))
-    (property "Value" "6pF" (id 1) (at 262.89 60.325 90))
+    (property "Value" "C" (id 1) (at 262.89 60.325 90))
     (property "Footprint" "Capacitor_SMD:C_0402_1005Metric" (id 2) (at 255.27 61.2648 0)
       (effects (font (size 1.27 1.27)) hide)
@@
     (in_bom yes) (on_board yes)
     (property "Reference" "R2" (id 0) (at 187.96 25.4 90))
-    (property "Value" "10K" (id 1) (at 187.96 27.94 90))
+    (property "Value" "R" (id 1) (at 187.96 27.94 90))
     (property "Footprint" "Resistor_SMD:R_0402_1005Metric" (id 2) (at 187.96 26.162 90)
       (effects (font (size 1.27 1.27)) hide)
@@
     (in_bom yes) (on_board yes)
     (property "Reference" "R3" (id 0) (at 238.76 80.01 90))
-    (property "Value" "10K" (id 1) (at 238.76 82.55 90))
+    (property "Value" "R" (id 1) (at 238.76 82.55 90))
     (property "Footprint" "Resistor_SMD:R_0402_1005Metric" (id 2) (at 238.76 80.772 90)
       (effects (font (size 1.27 1.27)) hide)
@@
     (in_bom yes) (on_board yes)
     (property "Reference" "C5" (id 0) (at 185.166 31.242 90))
-    (property "Value" "0.1uF" (id 1) (at 187.96 36.83 90))
+    (property "Value" "C" (id 1) (at 187.96 36.83 90))
     (property "Footprint" "Capacitor_SMD:C_0402_1005Metric" (id 2) (at 191.77 33.9852 0)
       (effects (font (size 1.27 1.27)) hide)
@@
     (in_bom yes) (on_board yes)
     (property "Reference" "C4" (id 0) (at 148.59 86.36 0))
-    (property "Value" "0.1uF" (id 1) (at 157.734 86.36 0))
+    (property "Value" "C" (id 1) (at 157.734 86.36 0))
     (property "Footprint" "Capacitor_SMD:C_0402_1005Metric" (id 2) (at 151.4348 90.17 0)
       (effects (font (size 1.27 1.27)) hide)
@@
     (in_bom yes) (on_board yes)
     (property "Reference" "C3" (id 0) (at 87.63 87.63 0))
-    (property "Value" "0.1uF" (id 1) (at 96.774 87.63 0))
+    (property "Value" "C" (id 1) (at 96.774 87.63 0))
     (property "Footprint" "Capacitor_SMD:C_0402_1005Metric" (id 2) (at 90.4748 91.44 0)
       (effects (font (size 1.27 1.27)) hide)
@@
     (in_bom yes) (on_board yes)
     (property "Reference" "R1" (id 0) (at 38.1 154.94 0))
-    (property "Value" "1K" (id 1) (at 33.02 154.94 0))
+    (property "Value" "R" (id 1) (at 33.02 154.94 0))
     (property "Footprint" "Resistor_SMD:R_0402_1005Metric" (id 2) (at 33.782 154.94 90)
       (effects (font (size 1.27 1.27)) hide)
@@
     (in_bom yes) (on_board yes)
     (property "Reference" "C11" (id 0) (at 261.874 71.628 90))
-    (property "Value" "6pF" (id 1) (at 262.89 67.945 90))
+    (property "Value" "C" (id 1) (at 262.89 67.945 90))
     (property "Footprint" "Capacitor_SMD:C_0402_1005Metric" (id 2) (at 255.27 68.8848 0)
       (effects (font (size 1.27 1.27)) hide)
@@
     (in_bom yes) (on_board yes)
     (property "Reference" "C6" (id 0) (at 230.505 107.95 0))
-    (property "Value" "1uF" (id 1) (at 227.965 105.41 0))
+    (property "Value" "C" (id 1) (at 227.965 105.41 0))
     (property "Footprint" "Capacitor_SMD:C_0402_1005Metric" (id 2) (at 233.3752 101.6 0)
       (effects (font (size 1.27 1.27)) hide)
@@
       (effects (font (size 1.27 1.27)) (justify left bottom))
     )
-    (property "Value" "1uF" (id 1) (at 49.53 35.56 0)
+    (property "Value" "CAP_0402" (id 1) (at 49.53 35.56 0)
       (effects (font (size 1.27 1.27)) (justify left bottom))
     )
-    (property "Footprint" "Capacitor_SMD:C_0402_1005Metric" (id 2) (at 50.8 36.83 0)
+    (property "Footprint" "Uinio:CAP_0402" (id 2) (at 50.8 36.83 0)
       (effects (font (size 1.27 1.27)) hide)
     )
@@
     (in_bom yes) (on_board yes)
     (property "Reference" "C9" (id 0) (at 246.126 93.472 90))
-    (property "Value" "0.1uF" (id 1) (at 253.238 93.472 90))
+    (property "Value" "C" (id 1) (at 253.238 93.472 90))
     (property "Footprint" "Capacitor_SMD:C_0402_1005Metric" (id 2) (at 252.73 92.4052 0)
       (effects (font (size 1.27 1.27)) hide)
@@
     (pin "2")
   )
-  (symbol (lib_name "USB_Type_C_6Pin_1") (lib_id "Uinio:USB_Type_C_6Pin") (at 87.63 148.59 0) (unit 1)
+  (symbol (lib_id "Uinio:USB_Type_C_6Pin") (at 87.63 148.59 0) (unit 1)
     (in_bom yes) (on_board yes)
     (property "Reference" "USB1" (id 0) (at 86.36 137.795 0))
@@
       (effects (font (size 1.27 1.27)) (justify left bottom))
     )
-    (property "Value" "1uF" (id 1) (at 85.09 36.83 0)
+    (property "Value" "CAP_0402" (id 1) (at 85.09 36.83 0)
       (effects (font (size 1.27 1.27)) (justify left bottom))
     )
-    (property "Footprint" "Capacitor_SMD:C_0402_1005Metric" (id 2) (at 86.36 38.1 0)
+    (property "Footprint" "Uinio:CAP_0402" (id 2) (at 86.36 38.1 0)
       (effects (font (size 1.27 1.27)) hide)
     )
@@
     (in_bom yes) (on_board yes)
     (property "Reference" "U1" (id 0) (at 73.914 38.862 0))
-    (property "Value" "ME6211C33M5G-N" (id 1) (at 73.66 53.34 0))
+    (property "Value" "ME6211" (id 1) (at 73.66 53.34 0))
     (property "Footprint" "Uinio:SOT-23-5_L3.0-W1.7-P0.95-LS2.8-BR" (id 2) (at 60.96 43.18 0)
       (effects (font (size 1.27 1.27)) hide)
@@
     (in_bom yes) (on_board yes)
     (property "Reference" "C8" (id 0) (at 238.125 107.95 0))
-    (property "Value" "0.1uF" (id 1) (at 245.11 105.41 0))
+    (property "Value" "C" (id 1) (at 245.11 105.41 0))
     (property "Footprint" "Capacitor_SMD:C_0402_1005Metric" (id 2) (at 240.9952 101.6 0)
       (effects (font (size 1.27 1.27)) hide)
@@
     )
     (path "/60560b20-5278-4de9-a5e2-fed3a53f08b4"
-      (reference "C1") (unit 1) (value "1uF") (footprint "Capacitor_SMD:C_0402_1005Metric")
+      (reference "C1") (unit 1) (value "CAP_0402") (footprint "Uinio:CAP_0402")
     )
     (path "/b5fedec1-4dc3-434f-a196-1e35f26eed3c"
-      (reference "C2") (unit 1) (value "1uF") (footprint "Capacitor_SMD:C_0402_1005Metric")
+      (reference "C2") (unit 1) (value "CAP_0402") (footprint "Uinio:CAP_0402")
     )
     (path "/450e9fbe-b5fb-4a9a-bff0-f14f6373f59c"
-      (reference "C3") (unit 1) (value "0.1uF") (footprint "Capacitor_SMD:C_0402_1005Metric")
+      (reference "C3") (unit 1) (value "C") (footprint "Capacitor_SMD:C_0402_1005Metric")
     )
     (path "/3ac80d50-3520-439d-b818-e8b1706d2c50"
-      (reference "C4") (unit 1) (value "0.1uF") (footprint "Capacitor_SMD:C_0402_1005Metric")
+      (reference "C4") (unit 1) (value "C") (footprint "Capacitor_SMD:C_0402_1005Metric")
     )
     (path "/336e24fa-e623-4dd7-85da-fa8081816864"
-      (reference "C5") (unit 1) (value "0.1uF") (footprint "Capacitor_SMD:C_0402_1005Metric")
+      (reference "C5") (unit 1) (value "C") (footprint "Capacitor_SMD:C_0402_1005Metric")
     )
     (path "/5706b301-f703-4c85-a59e-e955d05b4084"
-      (reference "C6") (unit 1) (value "1uF") (footprint "Capacitor_SMD:C_0402_1005Metric")
+      (reference "C6") (unit 1) (value "C") (footprint "Capacitor_SMD:C_0402_1005Metric")
     )
     (path "/0416ee8a-8799-47cf-9c7f-63d3a3f327e4"
-      (reference "C7") (unit 1) (value "0.1uF") (footprint "Capacitor_SMD:C_0402_1005Metric")
+      (reference "C7") (unit 1) (value "C") (footprint "Capacitor_SMD:C_0402_1005Metric")
     )
     (path "/eafae641-2814-4631-bc2a-0707f895595c"
-      (reference "C8") (unit 1) (value "0.1uF") (footprint "Capacitor_SMD:C_0402_1005Metric")
+      (reference "C8") (unit 1) (value "C") (footprint "Capacitor_SMD:C_0402_1005Metric")
     )
     (path "/6439d159-41c1-45b5-a4d6-02bcf2882093"
-      (reference "C9") (unit 1) (value "0.1uF") (footprint "Capacitor_SMD:C_0402_1005Metric")
+      (reference "C9") (unit 1) (value "C") (footprint "Capacitor_SMD:C_0402_1005Metric")
     )
     (path "/04927899-643a-465f-a90f-2fe0fcac3f7d"
-      (reference "C10") (unit 1) (value "6pF") (footprint "Capacitor_SMD:C_0402_1005Metric")
+      (reference "C10") (unit 1) (value "C") (footprint "Capacitor_SMD:C_0402_1005Metric")
     )
     (path "/4fa74506-c2c7-4363-ba60-ed462593bd01"
-      (reference "C11") (unit 1) (value "6pF") (footprint "Capacitor_SMD:C_0402_1005Metric")
+      (reference "C11") (unit 1) (value "C") (footprint "Capacitor_SMD:C_0402_1005Metric")
     )
     (path "/247e2303-24d7-4ed1-8e48-01c05cb88b4f"
@@
     )
     (path "/483d1138-1ab5-4212-90f2-9bef370560a2"
-      (reference "R1") (unit 1) (value "1K") (footprint "Resistor_SMD:R_0402_1005Metric")
+      (reference "R1") (unit 1) (value "R") (footprint "Resistor_SMD:R_0402_1005Metric")
     )
     (path "/0826aa88-c03d-4006-8191-9f916bbdd10b"
-      (reference "R2") (unit 1) (value "10K") (footprint "Resistor_SMD:R_0402_1005Metric")
+      (reference "R2") (unit 1) (value "R") (footprint "Resistor_SMD:R_0402_1005Metric")
     )
     (path "/0dc4dc38-298e-43a4-a369-891beafa0569"
-      (reference "R3") (unit 1) (value "10K") (footprint "Resistor_SMD:R_0402_1005Metric")
+      (reference "R3") (unit 1) (value "R") (footprint "Resistor_SMD:R_0402_1005Metric")
     )
     (path "/a26fb178-aeb6-4dfd-8d0f-683b1e6bca57"
@@
     )
     (path "/c781bc88-e38e-4e05-971f-4291248e0e6d"
-      (reference "U1") (unit 1) (value "ME6211C33M5G-N") (footprint "Uinio:SOT-23-5_L3.0-W1.7-P0.95-LS2.8-BR")
+      (reference "U1") (unit 1) (value "ME6211") (footprint "Uinio:SOT-23-5_L3.0-W1.7-P0.95-LS2.8-BR")
     )
     (path "/8ace1bf8-4c97-4b29-8087-2da24750bdd0"

Commit message: Update folders.
Parts:
- C1, C2: value CAP_0402 -> 1uF
- C10, C11: value C -> 6pF
- C3, C4, C5, C6, C7, C9: value C -> 0.1uF
- C8: value C -> 1uF
- D1: value LED -> Red LED
- R1: value R -> 1K
- R2, R3: value R -> 10K
Other:
- moved on the sheet: C2, R3
