File: UINIO-MCU-STM32L051K8.kicad_sch (KiCad schematic)
At the start: 26 parts, among them J1 Conn_01x14_Male, J2 Conn_01x14_Male, J3 Conn_01x04_Male, SW1 SW_Push, SW2 SW_Push, U1 ME6211, U2 W25Q128JVSSIQ, U3 STM32L051K8U6, Y1 FC135-32.768

Commit message: Release UINIO-MCU-STM32L051K8 version 3.1.0.
Parts:
- removed Y1: FC135-32.768, Uinio:CRYSTAL-FC135-32.768, symbol Uinio:FC135-32.768
- added Y1: Crystal-FC135-32.768, Uinio:CRYSTAL-FC135-32.768, symbol Uinio:Crystal-FC135-32.768
Connections:
- net at C10.2, U3.2 (PC14-OSC_IN): now also Y1.2 (GND)
- net at C11.2, U3.3 (PC15-OSC_OUT): now also Y1.1
Other:
- moved on the sheet: C6, C8, SW1

Commit message: Release UINIO-MCU-STM32L051K8 version 3.1.0.
Parts:
- C1, C2: footprint Uinio:CAP_0402 -> Capacitor_SMD:C_0402_1005Metric
Changed lines of the file:
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@@
       (effects (font (size 1.27 1.27)) (justify left bottom))
     )
-    (property "Footprint" "Uinio:CAP_0402" (id 2) (at 50.8 36.83 0)
+    (property "Footprint" "Capacitor_SMD:C_0402_1005Metric" (id 2) (at 50.8 36.83 0)
       (effects (font (size 1.27 1.27)) hide)
     )
@@
       (effects (font (size 1.27 1.27)) (justify left bottom))
     )
-    (property "Footprint" "Uinio:CAP_0402" (id 2) (at 86.36 36.83 0)
+    (property "Footprint" "Capacitor_SMD:C_0402_1005Metric" (id 2) (at 86.36 36.83 0)
       (effects (font (size 1.27 1.27)) hide)
     )
@@
     )
     (path "/60560b20-5278-4de9-a5e2-fed3a53f08b4"
-      (reference "C1") (unit 1) (value "1uF") (footprint "Uinio:CAP_0402")
+      (reference "C1") (unit 1) (value "1uF") (footprint "Capacitor_SMD:C_0402_1005Metric")
     )
     (path "/b5fedec1-4dc3-434f-a196-1e35f26eed3c"
-      (reference "C2") (unit 1) (value "1uF") (footprint "Uinio:CAP_0402")
+      (reference "C2") (unit 1) (value "1uF") (footprint "Capacitor_SMD:C_0402_1005Metric")
     )
     (path "/450e9fbe-b5fb-4a9a-bff0-f14f6373f59c"

Commit message: Release UINIO-MCU-STM32L051K8 version 3.2.0.
Connections:
- net VDD_3.3V: now also R1.2
- net VDD_5V: no longer R1.2
Other:
- moved on the sheet: C1, C2, D1, F1, R1, U1, USB1

Commit message: Update version.
Parts:
- removed J1, J2: Conn_01x14_Male, Connector_PinHeader_2.54mm:PinHeader_1x14_P2.54mm_Vertical, symbol Connector:Conn_01x14_Male
- removed J3: Conn_01x04_Male, Connector_PinHeader_2.54mm:PinHeader_1x04_P2.54mm_Vertical, symbol Connector:Conn_01x04_Male
- added J1, J2: Conn_01x14_Pin, Connector_PinHeader_2.54mm:PinHeader_1x14_P2.54mm_Vertical, symbol Connector:Conn_01x14_Pin
- added J3: Conn_01x04_Pin, Connector_PinHeader_2.54mm:PinHeader_1x04_P2.54mm_Vertical, symbol Connector:Conn_01x04_Pin
Connections:
- net GND: now also J2.2 (Pin_2), J2.4 (Pin_4), J3.4 (Pin_4)
- net NRST: now also J2.5 (Pin_5)
- net PA0: now also J1.1 (Pin_1)
- net PA1: now also J1.2 (Pin_2)
- net PA10: now also J1.11 (Pin_11)
- net PA11: now also J1.12 (Pin_12)
- net PA12: now also J1.13 (Pin_13)
- net PA13/SWDIO: now also J3.2 (Pin_2)
- net PA14/SWCLK: now also J3.3 (Pin_3)
- net PA15: now also J1.14 (Pin_14)
- net PA2: now also J1.3 (Pin_3)
- net PA3: now also J1.4 (Pin_4)
- net PA4/CS: now also J1.5 (Pin_5)
- net PA5/SCLK: now also J1.6 (Pin_6)
- net PA6/MISO: now also J1.7 (Pin_7)
- net PA7/MOSI: now also J1.8 (Pin_8)
- net PA8: now also J1.9 (Pin_9)
- net PA9: now also J1.10 (Pin_10)
- net PB0: now also J2.14 (Pin_14)
- net PB1: now also J2.13 (Pin_13)
- net PB2: now also J2.12 (Pin_12)
- net PB3: now also J2.11 (Pin_11)
- net PB4: now also J2.10 (Pin_10)
- net PB5: now also J2.9 (Pin_9)
- net PB6: now also J2.8 (Pin_8)
- net PB7: now also J2.7 (Pin_7)
- net PB8: now also J2.6 (Pin_6)
- net VDD_3.3V: now also J2.3 (Pin_3), J3.1 (Pin_1)
- net VDD_5V: now also J2.1 (Pin_1)
