File: UINIO-MCU-STM32L051K8U6.kicad_pcb (KiCad board)
At the start: 2 copper layers, 48.3 x 20.3 mm, 32 parts, among them J1 Conn_01x14_Pin, J2 Conn_01x14_Pin, J3 Conn_01x04_Pin, SW1 Boot选择按键, SW2 复位按键, U1 ME6211, U2 W25Q128JVSSIQ, U3 STM32L051K8U6, Y1 Crystal-FC135-32.768

Commit message: Release UINIO-MCU-STM32L051K8U6 version 3.3.0.
Other:
- board text added: "UINIO-MCU-STM32L051K8U6"
- board text removed: "UINIO-MCU-STM32L051K8"

Commit message: Release UINIO-MCU-STM32L051K8U6 version 3.3.1.
Parts:
- removed ? (x2): LOGO, LOGO
Other:
- board text added: "STM32L051K8U6"
- board text added: "Version 3.3.1"
- board text removed: "UINIO-MCU-STM32L051K8U6"
- board text removed: "Version 3.3.0"
