File: UINIO-MCU-STM32L051K8U6.kicad_pcb (KiCad board)
At the start: 2 copper layers, 48.3 x 20.3 mm, 30 parts, among them J1 Conn_01x14_Pin, J2 Conn_01x14_Pin, J3 Conn_01x04_Pin, SW1 Boot选择按键, SW2 复位按键, U1 ME6211, U2 W25Q128JVSSIQ, U3 STM32L051K8U6, Y1 Crystal-FC135-32.768

Commit message: Release UINIO-MCU-STM32L051K8U version 3.3.1.
Other:
- board text added: "UINIO-MCU-STM32L051K8U6"
- board text removed: "STM32L051K8U6"

Commit message: Release UINIO-MCU-STM32L051K8U6 version 3.3.2.
Routing:
- net /PA15: track 20.2 -> 18.5 mm
- net GND: vias 29 -> 43
Other:
- board text added: "Version 3.3.2"
- board text removed: "Version 3.3.1"

Commit message: Release UINIO-MCU-STM32L051K8U6 version 3.3.2.
Other:
- board text removed: "ARM"

Commit message: Release UINIO-MCU-STM32L051K8U6 version 3.3.2.
Routing:
- net GND: track 193.3 -> 191.1 mm, vias 43 -> 44
Other:
- outline, holes or cut-outs redrawn
